Commit message: posición palancas futbol
angulos de las palanacas de los servos corregidos en el urdf

File: install/futbol_robot/share/futbol_robot/urdf/futbol_robot.urdf (robot description, URDF)
Before this commit: robot futbol_robot, 6 links, 5 joints
Joints:
- joint servoder_joint: origin xyz=0.028374 0.093324 0.026131 rpy=-3.1416 -0.0020221 -1.5708 -> xyz=0.028374 0.093324 0.026131 rpy=-3.1416 -0.0020221 -1.7
- joint servoizq_joint: origin xyz=-0.029099 0.092707 0.026132 rpy=-3.1416 -0.0020221 -1.5708 -> xyz=-0.029099 0.092707 0.026132 rpy=-3.1416 -0.0020221 0.75
