Commit message: mejoras, muchas mejoras
codigo en esp32 con micro ros para sumo funciona, nuevo urdf para sumo funciona perfecto, en rviz se ven las referencias de los sensores, en gazebo se ve bien

File: install/sumo_robot/share/sumo_robot/urdf/sumo_robot.urdf (robot description, URDF)
Before this commit: robot sumo_robot, 4 links, 3 joints
Links:
- removed link Rueda_Derecha_Link
- removed link Rueda_Izquierda_Link
- added link ruedader_Link, mass 0.00900114044055008; collision mesh filename=package://sumo_robot/meshes/ruedader_Link.STL; visual mesh filename=package://sumo_robot/meshes/ruedader_Link.STL
- added link ruedaizq_Link, mass 0.00900114044055008; collision mesh filename=package://sumo_robot/meshes/ruedaizq_Link.STL; visual mesh filename=package://sumo_robot/meshes/ruedaizq_Link.STL
- added link vl53_centro, mass 1.65901982165976E-06; collision mesh filename=package://sumo_robot/meshes/sensorcentro_Link.STL; visual mesh filename=package://sumo_robot/meshes/sensorcentro_Link.STL
- added link vl53_der, mass 1.65901978024444E-06; collision mesh filename=package://sumo_robot/meshes/sensorder_Link.STL; visual mesh filename=package://sumo_robot/meshes/sensorder_Link.STL
- added link vl53_izq, mass 1.65901978015762E-06; collision mesh filename=package://sumo_robot/meshes/sensorizq_Link.STL; visual mesh filename=package://sumo_robot/meshes/sensorizq_Link.STL
- link base_link: mass 0.249564590974204 -> 0.229572965520933
Joints:
- removed joint Rueda_Derecha_joint
- removed joint Rueda_Izquierda_joint
- added joint ruedader_joint: type continuous, parent base_link, child ruedader_Link, origin xyz=0.0036812 -0.0465 0.013458 rpy=1.5708 0 0, axis 0 0 -1, limit effort=50 velocity=50
- added joint ruedaizq_joint: type continuous, parent base_link, child ruedaizq_Link, origin xyz=0.0036812 0.0465 0.013458 rpy=1.5708 0 3.1416, axis 0 0 -1, limit effort=50 velocity=50
- added joint vl53_centro_joint: type fixed, parent base_link, child vl53_centro, origin xyz=0.067284 0.00056819 0.051217 rpy=1.7453 0 1.5708
- added joint vl53_der_joint: type fixed, parent base_link, child vl53_der, origin xyz=0.062963 -0.029939 0.051217 rpy=1.7453 0 1.309
- added joint vl53_izq_joint: type fixed, parent base_link, child vl53_izq, origin xyz=0.062889 0.030215 0.051217 rpy=1.7453 0 1.8326
- joint base_footprint_joint: origin xyz=0 0 0.081 rpy=1.5707963 0 0 -> xyz=0 0 0.0075 rpy=0 0 0

File: src/sumo_robot/urdf/sumo_robot.urdf (robot description, URDF)
Before this commit: robot sumo_robot, 4 links, 3 joints
Links:
- removed link Rueda_Derecha_Link
- removed link Rueda_Izquierda_Link
- added link ruedader_Link, mass 0.00900114044055008; collision mesh filename=package://sumo_robot/meshes/ruedader_Link.STL; visual mesh filename=package://sumo_robot/meshes/ruedader_Link.STL
- added link ruedaizq_Link, mass 0.00900114044055008; collision mesh filename=package://sumo_robot/meshes/ruedaizq_Link.STL; visual mesh filename=package://sumo_robot/meshes/ruedaizq_Link.STL
- added link vl53_centro, mass 1.65901982165976E-06; collision mesh filename=package://sumo_robot/meshes/sensorcentro_Link.STL; visual mesh filename=package://sumo_robot/meshes/sensorcentro_Link.STL
- added link vl53_der, mass 1.65901978024444E-06; collision mesh filename=package://sumo_robot/meshes/sensorder_Link.STL; visual mesh filename=package://sumo_robot/meshes/sensorder_Link.STL
- added link vl53_izq, mass 1.65901978015762E-06; collision mesh filename=package://sumo_robot/meshes/sensorizq_Link.STL; visual mesh filename=package://sumo_robot/meshes/sensorizq_Link.STL
- link base_link: mass 0.249564590974204 -> 0.229572965520933
Joints:
- removed joint Rueda_Derecha_joint
- removed joint Rueda_Izquierda_joint
- added joint ruedader_joint: type continuous, parent base_link, child ruedader_Link, origin xyz=0.0036812 -0.0465 0.013458 rpy=1.5708 0 0, axis 0 0 -1, limit effort=50 velocity=50
- added joint ruedaizq_joint: type continuous, parent base_link, child ruedaizq_Link, origin xyz=0.0036812 0.0465 0.013458 rpy=1.5708 0 3.1416, axis 0 0 -1, limit effort=50 velocity=50
- added joint vl53_centro_joint: type fixed, parent base_link, child vl53_centro, origin xyz=0.067284 0.00056819 0.051217 rpy=1.7453 0 1.5708
- added joint vl53_der_joint: type fixed, parent base_link, child vl53_der, origin xyz=0.062963 -0.029939 0.051217 rpy=1.7453 0 1.309
- added joint vl53_izq_joint: type fixed, parent base_link, child vl53_izq, origin xyz=0.062889 0.030215 0.051217 rpy=1.7453 0 1.8326
- joint base_footprint_joint: origin xyz=0 0 0.081 rpy=1.5707963 0 0 -> xyz=0 0 0.0075 rpy=0 0 0

Commit message: todo funcionando, falta el giro en gazebo

File: install/sumo_robot/share/sumo_robot/urdf/sumo_robot.urdf (robot description, URDF)
Before this commit: robot sumo_robot, 7 links, 6 joints
Joints:
- joint vl53_centro_joint: origin xyz=0.067284 0.00056819 0.051217 rpy=1.7453 0 1.5708 -> xyz=0.067284 0.00056819 0.051217 rpy=1.7453 0 0
- joint vl53_der_joint: origin xyz=0.062963 -0.029939 0.051217 rpy=1.7453 0 1.309 -> xyz=0.062963 -0.029939 0.051217 rpy=1.7453 0 -0.2618
- joint vl53_izq_joint: origin xyz=0.062889 0.030215 0.051217 rpy=1.7453 0 1.8326 -> xyz=0.062889 0.030215 0.051217 rpy=1.7453 0 0.2618
