Commit message: Ultimos cambios finales

File: src/futbol_robot/urdf/futbol_robot.urdf (robot description, URDF)
Before this commit: robot futbol_robot, 6 links, 5 joints
Joints:
- joint ruedaizq_joint: axis 0 0 -1 -> 0 0 1

File: src/sumo_robot/urdf/sumo_robot.urdf (robot description, URDF)
Before this commit: robot sumo_robot, 7 links, 6 joints
Joints:
- joint ruedaizq_joint: axis 0 0 -1 -> 0 0 1
